File: _saved_oshw2018badgeprototype.sch (KiCad schematic (older format))
At the start: 59 parts, among them J1 Conn_02x03_Top_Bottom, J2 105162-0001, Q2 Q_NMOS_GSD, SW1 SW_Push, T1 TEST_1P, T2 TEST_1P, T3 TEST_1P, T4 TEST_1P, T5 TEST_1P, T6 TEST_1P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

Commit message: Improved silkscreen Artwork and added Testpoints
Parts:
- renumbered BAT to BAT1, EN to EN1, GND to GND1, RXD to RXD1, TXD to TXD1
Changed lines of the file:
@@
 EN
 $Comp
-L oshw2018badgeprototype-rescue:GND #PWR?
+L oshw2018badgeprototype-rescue:GND #PWR0101
 U 1 1 5B662290
 P 2650 -800
-F 0 "#PWR?" H 2650 -1050 50  0001 C CNN
+F 0 "#PWR0101" H 2650 -1050 50  0001 C CNN
 F 1 "GND" H 2650 -950 50  0000 C CNN
 F 2 "" H 2650 -800 50  0001 C CNN
@@
 $EndComp
 $Comp
-L oshw2018badgeprototype-rescue:+3V3 #PWR?
+L oshw2018badgeprototype-rescue:+3V3 #PWR0102
 U 1 1 5B6628B9
 P 2650 -1000
-F 0 "#PWR?" H 2650 -1150 50  0001 C CNN
+F 0 "#PWR0102" H 2650 -1150 50  0001 C CNN
 F 1 "+3V3" H 2650 -860 50  0000 C CNN
 F 2 "" H 2650 -1000 50  0001 C CNN
@@
 	6200 5950 6350 5950
 $Comp
-L Connector:TestPoint EN
+L Connector:TestPoint EN1
 U 1 1 5B67725A
 P 1850 -650
-F 0 "EN" V 1850 -463 50  0000 L CNN
+F 0 "EN1" V 1850 -463 50  0000 L CNN
 F 1 "TestPoint" V 1895 -462 50  0001 L CNN
 F 2 "test_point:test_point" H 2050 -650 50  0001 C CNN
@@
 $EndComp
 $Comp
-L Connector:TestPoint TXD
+L Connector:TestPoint TXD1
 U 1 1 5B6772FE
 P 1850 -550
-F 0 "TXD" V 1850 -363 50  0000 L CNN
+F 0 "TXD1" V 1850 -363 50  0000 L CNN
 F 1 "TestPoint" V 1895 -362 50  0001 L CNN
 F 2 "test_point:test_point" H 2050 -550 50  0001 C CNN
@@
 $EndComp
 $Comp
-L Connector:TestPoint RXD
+L Connector:TestPoint RXD1
 U 1 1 5B67737E
 P 1850 -450
-F 0 "RXD" V 1850 -263 50  0000 L CNN
+F 0 "RXD1" V 1850 -263 50  0000 L CNN
 F 1 "TestPoint" V 1895 -262 50  0001 L CNN
 F 2 "test_point:test_point" H 2050 -450 50  0001 C CNN
@@
 $EndComp
 $Comp
-L Connector:TestPoint BAT
+L Connector:TestPoint BAT1
 U 1 1 5B677488
 P 1850 -250
-F 0 "BAT" V 1850 -62 50  0000 L CNN
+F 0 "BAT1" V 1850 -62 50  0000 L CNN
 F 1 "TestPoint" V 1895 -62 50  0001 L CNN
 F 2 "test_point:test_point" H 2050 -250 50  0001 C CNN
@@
 $EndComp
 $Comp
-L Connector:TestPoint GND
+L Connector:TestPoint GND1
 U 1 1 5B677C91
 P 2600 -800
-F 0 "GND" V 2703 -726 50  0000 C CNN
+F 0 "GND1" V 2703 -726 50  0000 C CNN
 F 1 "TestPoint" V 2645 -612 50  0001 L CNN
 F 2 "test_point:test_point" H 2800 -800 50  0001 C CNN
